File: hardware/OpenAirStation-V0-Draft/OpenAirScope.kicad_pcb (KiCad board)
At the start: 4 copper layers, 100 x 75 mm, 282 parts, among them J1 USB_C_Receptacle_USB2.0_16P, J10 S5B-ZR_LF__SN_, J11 Micro_SD_Card, J13 Conn_01x07_Pin, J14 Conn_01x08_Pin, J2 S2B-PH-K-S_LF__SN_, J3 Conn_ST_STDC14, J4 Conn_01x08_Pin, J5 Conn_01x08_Pin, J6 RFPC-SMA27-F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

Commit message: v0.2
Routing:
- net +3V3P_MCU: track 196.6 -> 194.7 mm
Other:
- board text added: "OpenAirScope"
- board text removed: "OpenAirStation"
