File: hardware/OpenAirStation-V0-Draft/OpenAirScope.kicad_pcb (KiCad board)
At the start: 4 copper layers, 100 x 75 mm, 282 parts, among them J1 USB_C_Receptacle_USB2.0_16P, J10 S5B-ZR_LF__SN_, J11 Micro_SD_Card, J13 Conn_01x07_Pin, J14 Conn_01x08_Pin, J2 S2B-PH-K-S_LF__SN_, J3 Conn_ST_STDC14, J4 Conn_01x08_Pin, J5 Conn_01x08_Pin, J6 RFPC-SMA27-F, J7 Conn_01x07_Pin, J8 Screw_Terminal_01x02, J9 Screw_Terminal_01x02, Q1 BC817, Q3 BC817, Q4 BC817, Q5 BC817, Q6 BC817, Q7 BC817, Q8 BC817, SW3 SW_Push, SW4 SW_Push, SW5 SW_Push, U1 MCP73871, U10 MAX3485, U11 SGP41-D-R4, U12 SCD40-D-R2, U13 LTR-303ALS-01, U14 CM1624, U15 DS3231M, U2 TPD2E2U06DCK, U3 TPS61023DRLT, U4 LD39150DT33-R, U5 STM32H743ZITx, U6 M95256-WMN6P, U7 ESP32-C3-WROOM-02, U8 RAK3172, U9 SN65HVD230

Commit message: v0.3
Other:
- board text added: "DESIGN NOTE: THIS PCB IS PROVIDED AS A REFERENCE DESIGN. GND REFERENCE PLANE IMPLEMENTATION IS PENDING AND SHALL BE INCLUDED IN THE FINAL DESIGN."
- board text added: "GND REFERENCE PLANE SHALL BE ADDED."
