File: hardware/OpenAirStation-V0-Draft/Conn.kicad_sch (KiCad schematic)
At the start: 58 parts, among them J15 JAE_SIM_Card_SF72S006, J4 Conn_01x08_Pin, J5 Conn_01x08_Pin, J6 RFPC-SMA27-F, J7 Conn_01x07_Pin, J8 Screw_Terminal_01x02, J9 Screw_Terminal_01x02, U10 MAX3485, U16 BC66, U7 ESP32-C3-WROOM-02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

Commit message: esp
Parts:
- C56: now not fitted
Changed lines of the file:
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@@
 		(in_bom yes)
 		(on_board yes)
-		(dnp no)
+		(dnp yes)
 		(fields_autoplaced yes)
 		(property "Reference" "C56"

Commit message: v0.2
Changed lines of the file:
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@@
 		)
 		(property "Datasheet" "http://www.ti.com/lit/ds/symlink/sn65hvd230.pdf"
-			(at 335.534 249.682 0)
+			(at 330.454 244.856 0)
 			(effects
 				(font
@@
 		)
 		(property "Datasheet" "https://datasheets.maximintegrated.com/en/ds/MAX3483-MAX3491.pdf"
-			(at 358.902 264.668 0)
+			(at 340.868 246.888 0)
 			(effects
 				(font

Commit message: v0.3
Parts:
- C53, C54: value ~ -> (none)
