File: hardware/OpenAirStation-V0-Draft/OpenAirScope_N.kicad_sch (KiCad schematic)
At the start: 0 parts

Commit message: v0.2
Changed lines of the file:
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@@
 		(effects
 			(font
-				(face "BankGothic Lt BT")
-				(size 5.08 5.08)
-				(bold yes)
-			)
-		)
-	)
-	(text "SENS\n"
-		(exclude_from_sim no)
-		(at 113.1794 128.5312 0)
-		(effects
-			(font
-				(face "BankGothic Lt BT")
+				(face "Arial")
 				(size 5.08 5.08)
 				(bold yes)
@@
 		(effects
 			(font
-				(face "BankGothic Lt BT")
+				(face "Arial")
 				(size 5.08 5.08)
 				(bold yes)
@@
 	(text "SENS\n"
 		(exclude_from_sim no)
-		(at 112.9656 142.322 0)
+		(at 113.538 129.54 0)
 		(effects
 			(font
-				(face "BankGothic Lt BT")
+				(face "Arial")
 				(size 5.08 5.08)
 				(bold yes)
@@
 		(effects
 			(font
-				(face "BankGothic Lt BT")
+				(face "Arial")
 				(size 5.08 5.08)
 				(bold yes)
@@
 		(effects
 			(font
-				(face "BankGothic Lt BT")
+				(face "Arial")
 				(size 5.08 5.08)
 				(bold yes)
@@
 		(effects
 			(font
-				(face "BankGothic Lt BT")
+				(face "Arial")
 				(size 5.08 5.08)
 				(bold yes)
@@
 		(effects
 			(font
-				(face "BankGothic Lt BT")
+				(face "Arial")
+				(size 5.08 5.08)
+				(bold yes)
+			)
+		)
+	)
+	(text "SENS\n"
+		(exclude_from_sim no)
+		(at 114.046 116.078 0)
+		(effects
+			(font
+				(face "Arial")
 				(size 5.08 5.08)
 				(bold yes)
@@
 		(effects
 			(font
-				(face "BankGothic Lt BT")
+				(face "Arial")
 				(size 5.08 5.08)
 				(bold yes)
@@
 		(effects
 			(font
-				(face "BankGothic Lt BT")
+				(face "Arial")
+				(size 5.08 5.08)
+				(bold yes)
+			)
+		)
+	)
+	(text "SENS\n"
+		(exclude_from_sim no)
+		(at 113.284 143.51 0)
+		(effects
+			(font
+				(face "Arial")
 				(size 5.08 5.08)
 				(bold yes)
@@
 		(effects
 			(font
-				(face "BankGothic Lt BT")
-				(size 5.08 5.08)
-				(bold yes)
-			)
-		)
-	)
-	(text "SENS\n"
-		(exclude_from_sim no)
-		(at 113.284 114.808 0)
-		(effects
-			(font
-				(face "BankGothic Lt BT")
+				(face "Arial")
 				(size 5.08 5.08)
 				(bold yes)
@@
 		(effects
 			(font
-				(face "BankGothic Lt BT")
+				(face "Arial")
 				(size 5.08 5.08)
 				(bold yes)
@@
 		(effects
 			(font
-				(face "BankGothic Lt BT")
+				(face "Arial")
 				(size 5.08 5.08)
 				(bold yes)
