File: hardware/OpenAirStation-V0-Draft/Power.kicad_sch (KiCad schematic)
At the start: 47 parts, among them J1 USB_C_Receptacle_USB2.0_16P, J2 S2B-PH-K-S_LF__SN_, U1 MCP73871, U2 TPD2E2U06DCK, U3 TPS61023DRLT, U4 LD39150DT33-R

Commit message: v0.3
Parts:
- J2: DESCRIPTION Connector Header Through Hole, Right Angle 2 position -> (none)
