File: hardware/OpenAirStation-V0-Draft/untitled.kicad_sch (KiCad schematic)
At the start: 77 parts, among them Q3 BC817, Q4 BC817, Q5 BC817, Q6 BC817, Q7 BC817, Q8 BC817, SW3 SW_Push, SW4 SW_Push, SW5 SW_Push

Commit message: v0
Parts:
- removed FID1, FID10, FID2, FID3, FID4, FID5, FID6, FID7, FID8, FID9: Fiducial, Fiducial:Fiducial_1mm_Mask2mm, symbol Mechanical:Fiducial
